Commit message: ugv_a: add Ranger model and Sensor model(airy and D435i models)

File: sensor_kit/ugv_a_sensor_kit_launch/ugv_a_sensor_kit_description/sensor/camera/urdf/d435i_camera.xacro (robot description, xacro)
@@ -1,5 +1,5 @@
 <?xml version="1.0"?>
 <robot xmlns:xacro="http://ros.org/wiki/xacro">
-  <xacro:macro name="monocular_camera_macro" params="name parent namespace x y z roll pitch yaw fps width height fov">
+  <xacro:macro name="d435i_camera_macro" params="name parent namespace x y z roll pitch yaw fps width height fov">
     <xacro:property name="sensor_box" value="0.05"/>
     <xacro:property name="mass" value="0.1"/>
@@ -10,9 +10,9 @@
     </joint>
     <link name="${name}_link">
-      <visual>
+       <visual>
         <geometry>
-          <box size="${sensor_box} ${sensor_box} ${sensor_box}"/>
+          <mesh filename="package://ugv_a_sensor_kit_description/sensor/camera/meshes/d435.dae" scale="1 1 1"/>
         </geometry>
-        <origin rpy="0 0 0" xyz="0 0 0"/>
+        <origin rpy="${pi/2} 0 ${pi/2}" xyz="0.0125 0 0"/>
         <material name="red">
           <color rgba="1.0 0.0 0.0 1.0"/>

File: sensor_kit/ugv_a_sensor_kit_launch/ugv_a_sensor_kit_description/urdf/sensor_kit.xacro (robot description, xacro)
@@ -2,6 +2,6 @@
 <robot xmlns:xacro="http://ros.org/wiki/xacro">
   <xacro:macro name="sensor_kit_macro" params="parent x y z roll pitch yaw">
-    <xacro:include filename="$(find ugv_a_sensor_kit_description)/sensor/vls/urdf/VLS-128.urdf.xacro"/>
-    <xacro:include filename="$(find ugv_a_sensor_kit_description)/sensor/camera/urdf/monocular_camera.xacro"/>
+    <xacro:include filename="$(find ugv_a_sensor_kit_description)/sensor/airy/urdf/airy.urdf.xacro"/>
+    <xacro:include filename="$(find ugv_a_sensor_kit_description)/sensor/camera/urdf/d435i_camera.xacro"/>
     <xacro:include filename="$(find ugv_a_sensor_kit_description)/sensor/imu/urdf/imu.xacro"/>
     <xacro:arg name="gpu" default="false"/>
@@ -19,5 +19,5 @@
     <xacro:property name="calibration" value="${xacro.load_yaml('$(arg config_dir)/sensor_kit_calibration.yaml')}"/>
     <!-- lidar -->
-    <xacro:VLS-128 parent="sensor_kit_base_link" name="rs_airy_top" topic="/points_raw" hz="10" samples="220" gpu="$(arg gpu)">
+    <xacro:Airy parent="sensor_kit_base_link" name="rs_airy_top" topic="/points_raw" hz="10" gpu="$(arg gpu)">
       <origin
         xyz="${calibration['sensor_kit_base_link']['rs_airy_top_base_link']['x']}
@@ -28,7 +28,7 @@
              ${calibration['sensor_kit_base_link']['rs_airy_top_base_link']['yaw']}"
       />
-    </xacro:VLS-128>
+    </xacro:Airy>
     <!-- camera -->
-    <xacro:monocular_camera_macro
+    <xacro:d435i_camera_macro
       name="d435i/camera"
       parent="sensor_kit_base_link"

File: vehicle/ugv_a_vehicle_launch/ugv_a_vehicle_description/urdf/vehicle.xacro (robot description, xacro)
@@ -5,8 +5,37 @@
   <!-- vehicle body -->
   <link name="base_link">
+    <!-- body: mesh origin is the top surface, deck height 0.345 -->
     <visual>
-      <origin xyz="${vehicle_info['/**']['ros__parameters']['wheel_base']/2.0} 0 0" rpy="${pi/2.0} 0 ${pi}"/>
+      <origin xyz="0 0 0.345" rpy="0 0 0"/>
       <geometry>
-        <mesh filename="package://ugv_a_vehicle_description/mesh/lexus.dae" scale="1 1 1"/>
+        <mesh filename="package://ugv_a_vehicle_description/mesh/ranger_base.dae" scale="1 1 1"/>
+      </geometry>
+    </visual>
+    <!-- front left wheel -->
+    <visual>
+      <origin xyz="${vehicle_info['/**']['ros__parameters']['wheel_base']} ${vehicle_info['/**']['ros__parameters']['wheel_tread']/2.0} ${vehicle_info['/**']['ros__parameters']['wheel_radius']}" rpy="0 0 0"/>
+      <geometry>
+        <mesh filename="package://ugv_a_vehicle_description/mesh/wheel_v3.dae" scale="14.1 10.6 14.1"/>
+      </geometry>
+    </visual>
+    <!-- front right wheel -->
+    <visual>
+      <origin xyz="${vehicle_info['/**']['ros__parameters']['wheel_base']} ${-vehicle_info['/**']['ros__parameters']['wheel_tread']/2.0} ${vehicle_info['/**']['ros__parameters']['wheel_radius']}" rpy="0 0 ${pi}"/>
+      <geometry>
+        <mesh filename="package://ugv_a_vehicle_description/mesh/wheel_v3.dae" scale="14.1 10.6 14.1"/>
+      </geometry>
+    </visual>
+    <!-- rear left wheel -->
+    <visual>
+      <origin xyz="${-vehicle_info['/**']['ros__parameters']['wheel_base']} ${vehicle_info['/**']['ros__parameters']['wheel_tread']/2.0} ${vehicle_info['/**']['ros__parameters']['wheel_radius']}" rpy="0 0 0"/>
+      <geometry>
+        <mesh filename="package://ugv_a_vehicle_description/mesh/wheel_v3.dae" scale="14.1 10.6 14.1"/>
+      </geometry>
+    </visual>
+    <!-- rear right wheel -->
+    <visual>
+      <origin xyz="${-vehicle_info['/**']['ros__parameters']['wheel_base']} ${-vehicle_info['/**']['ros__parameters']['wheel_tread']/2.0} ${vehicle_info['/**']['ros__parameters']['wheel_radius']}" rpy="0 0 ${pi}"/>
+      <geometry>
+        <mesh filename="package://ugv_a_vehicle_description/mesh/wheel_v3.dae" scale="14.1 10.6 14.1"/>
       </geometry>
     </visual>
