Commit message: ugv_a: use Airy driver (ugv_airy_driver) for lidar and IMU

File: sensor_kit/ugv_a_sensor_kit_launch/ugv_a_sensor_kit_description/sensor/airy/urdf/airy.urdf.xacro (robot description, xacro)
@@ -41,5 +41,5 @@
     <!-- TODO: set to the point cloud origin height from the Airy User Guide (placeholder: half height) -->
     <joint name="${name}_base_scan_joint" type="fixed">
-      <origin xyz="0 0 0.0315" rpy="0 0 0"/>
+      <origin xyz="0 0 0" rpy="0 0 0"/>
       <parent link="${name}_base_link"/>
       <child link="${name}"/>
